Commit message: added models provided by Anastasia

File: urdf/chair.urdf (robot description, URDF)
Before this commit: robot chair, 1 links, 0 joints
Links:
- removed link base_chair
- added link back_support
- added link base_link
- added link chair; collision box size=0.5 0.5 0.5; visual mesh filename=package://meshes/chair/chair.dae
- added link left_handle
- added link leg_fl
- added link leg_fr
- added link leg_rl
- added link leg_rr
- added link right_handle
Joints:
- added joint back_joint: type fixed, parent chair, child back_support
- added joint base: type fixed, parent base_link, child chair
- added joint leg_fl_joint: type fixed, parent chair, child leg_fl
- added joint leg_fr_joint: type fixed, parent chair, child leg_fr
- added joint leg_rl_joint: type fixed, parent chair, child leg_rl
- added joint leg_rr_joint: type fixed, parent chair, child leg_rr
- added joint lhandle_joint: type fixed, parent chair, child left_handle
- added joint rhandle_joint: type fixed, parent chair, child right_handle

File: urdf/table.urdf (robot description, URDF)
Before this commit: robot table, 1 links, 0 joints
Links:
- link base_table: geometry collision box size=1.6 0.7 0.7; visual mesh filename=package://meshes/table/table.stl
