Commit message: Changed urdf files from Anastasia to plot correctly in rviz2, with corresponding launch files

File: objects_descriptions/urdf/table.urdf.xacro (robot description, xacro)
@@ -1,11 +1,11 @@
 <?xml version="1.0"?>
 <robot name="table" xmlns:xacro="http://wiki.ros.org/xacro">
-  <xacro:arg name="prefix" default="table_"/>
-  <xacro:arg name="connected_to" default=""/>
-  <xacro:arg name="xyz" default="'0 0 0'"/>
-  <xacro:arg name="rpy" default="'0 0 0'"/>
-  <xacro:arg name="mass" default="3.0"/>
-  <xacro:include filename="$(find objects_descriptions)/urdf/table.xacro"/>
-  <xacro:open_box prefix="$(arg prefix)" connected_to="$(arg connected_to)" xyz="$(arg xyz)" rpy="$(arg rpy)"
-                  mass="$(arg mass)"/>
+    <xacro:arg name="prefix" default="table_"/>
+    <xacro:arg name="connected_to" default=""/>
+    <xacro:arg name="xyz" default="'0 0 0'"/>
+    <xacro:arg name="rpy" default="'0 0 0'"/>
+    <xacro:arg name="mass" default="3.0"/>
+    <xacro:include filename="$(find objects_descriptions)/urdf/table.xacro"/>
+    <xacro:table prefix="$(arg prefix)" connected_to="$(arg connected_to)" xyz="$(arg xyz)" rpy="$(arg rpy)"
+                 mass="$(arg mass)"/>
 </robot>

File: objects_descriptions/urdf/wheelchair.xacro (robot description, xacro)
@@ -1,9 +1,6 @@
 <?xml version="1.0"?>
-<robot name="table_sim" xmlns:xacro="http://wiki.ros.org/xacro">
-    <xacro:macro name="table"
-                 params="prefix='table_' connected_to:='' xyz:='0 0 0' rpy:='0 0 0' mass=3.0">
-        <material name="Shape.003">
-            <color rgba="0.33 0.24 0.15 1"/>
-        </material>
+<robot name="wheelchair_sim" xmlns:xacro="http://wiki.ros.org/xacro">
+    <xacro:macro name="wheelchair"
+                 params="prefix='wheelchair_' connected_to:='' xyz:='0 0 0' rpy:='0 0 0' mass=3.0">
         <xacro:if value="${connected_to == ''}">
             <link name="world"/>
@@ -19,18 +16,21 @@
         <joint name="${prefix}base_to_${base_frame_name}" type="fixed">
             <parent link="${base_frame_name}"/>
-            <child link="${prefix}main_link"/>
+            <child link="${prefix}base_link"/>
             <origin rpy="${rpy}" xyz="${xyz}"/>
         </joint>
-        <link name="${prefix}main_link">
+        <link name="${prefix}base_link"/>
+        <joint name="${prefix}base" type="fixed">
+            <parent link="${prefix}base_link"/>
+            <child link="${prefix}chair"/>
+        </joint>
+        <link name="${prefix}chair">
             <visual>
                 <geometry>
-                    <mesh filename="package://objects_descriptions/meshes/table/table.stl"/>
+                    <mesh filename="package://objects_descriptions/meshes/wheelchair/wheelchair.dae"/>
                 </geometry>
-                <material name="Shape.003"/>
             </visual>
             <collision>
-                <origin xyz="0 0.18 0.4" rpy="0 0 0"/>
                 <geometry>
-                    <box size="1.6 0.7 0.7"/>
+                    <box size="0.5 0.5 0.5"/>
                 </geometry>
             </collision>

Commit message: commented fixed joint to get rid of jumpy behaviour

File: objects_descriptions/urdf/table.urdf.xacro (robot description, xacro)
@@ -5,5 +5,5 @@
     <xacro:arg name="xyz" default="'0 0 0'"/>
     <xacro:arg name="rpy" default="'0 0 0'"/>
-    <xacro:arg name="mass" default="3.0"/>
+    <xacro:arg name="mass" default="8.0"/>
     <xacro:include filename="$(find objects_descriptions)/urdf/table.xacro"/>
     <xacro:table prefix="$(arg prefix)" connected_to="$(arg connected_to)" xyz="$(arg xyz)" rpy="$(arg rpy)"

File: objects_descriptions/urdf/table.xacro (robot description, xacro)
@@ -6,20 +6,20 @@
             <color rgba="0.33 0.24 0.15 1"/>
         </material>
-        <xacro:if value="${connected_to == ''}">
-            <link name="world"/>
-            <xacro:property name="base_frame_name" value="world"/>
-        </xacro:if>
-        <xacro:unless value="${connected_to == ''}">
-            <xacro:property name="base_frame_name" value="${connected_to}"/>
-        </xacro:unless>
-        <xacro:if value="${connected_to == 'odom'}">
-            <link name="odom"/>
-            <xacro:property name="base_frame_name" value="odom"/>
-        </xacro:if>
-        <joint name="${prefix}base_to_${base_frame_name}" type="fixed">
-            <parent link="${base_frame_name}"/>
-            <child link="${prefix}main_link"/>
-            <origin rpy="${rpy}" xyz="${xyz}"/>
-        </joint>
+<!--        <xacro:if value="${connected_to == ''}">-->
+<!--            <link name="world"/>-->
+<!--            <xacro:property name="base_frame_name" value="world"/>-->
+<!--        </xacro:if>-->
+<!--        <xacro:unless value="${connected_to == ''}">-->
+<!--            <xacro:property name="base_frame_name" value="${connected_to}"/>-->
+<!--        </xacro:unless>-->
+<!--        <xacro:if value="${connected_to == 'odom'}">-->
+<!--            <link name="odom"/>-->
+<!--            <xacro:property name="base_frame_name" value="odom"/>-->
+<!--        </xacro:if>-->
+<!--        <joint name="${prefix}base_to_${base_frame_name}" type="fixed">-->
+<!--            <parent link="${base_frame_name}"/>-->
+<!--            <child link="${prefix}main_link"/>-->
+<!--            <origin rpy="${rpy}" xyz="${xyz}"/>-->
+<!--        </joint>-->
         <link name="${prefix}main_link">
             <visual>
