Commit message: Created multiple publishers to change the position of the models, removed macro to link to world

File: objects_descriptions/urdf/chair.xacro (robot description, xacro)
@@ -3,20 +3,20 @@
     <xacro:macro name="chair"
                  params="prefix='chair_' connected_to:='' xyz:='0 0 0' rpy:='0 0 0' mass=2.0">
-        <xacro:if value="${connected_to == ''}">
-            <link name="world"/>
-            <xacro:property name="base_frame_name" value="world"/>
-        </xacro:if>
-        <xacro:unless value="${connected_to == ''}">
-            <xacro:property name="base_frame_name" value="${connected_to}"/>
-        </xacro:unless>
-        <xacro:if value="${connected_to == 'odom'}">
-            <link name="odom"/>
-            <xacro:property name="base_frame_name" value="odom"/>
-        </xacro:if>
-        <joint name="${prefix}base_to_${base_frame_name}" type="fixed">
-            <parent link="${base_frame_name}"/>
-            <child link="${prefix}base_link"/>
-            <origin rpy="${rpy}" xyz="${xyz}"/>
-        </joint>
+<!--        <xacro:if value="${connected_to == ''}">-->
+<!--            <link name="world"/>-->
+<!--            <xacro:property name="base_frame_name" value="world"/>-->
+<!--        </xacro:if>-->
+<!--        <xacro:unless value="${connected_to == ''}">-->
+<!--            <xacro:property name="base_frame_name" value="${connected_to}"/>-->
+<!--        </xacro:unless>-->
+<!--        <xacro:if value="${connected_to == 'odom'}">-->
+<!--            <link name="odom"/>-->
+<!--            <xacro:property name="base_frame_name" value="odom"/>-->
+<!--        </xacro:if>-->
+<!--        <joint name="${prefix}base_to_${base_frame_name}" type="fixed">-->
+<!--            <parent link="${base_frame_name}"/>-->
+<!--            <child link="${prefix}base_link"/>-->
+<!--            <origin rpy="${rpy}" xyz="${xyz}"/>-->
+<!--        </joint>-->
         <link name="${prefix}base_link"/>
         <joint name="${prefix}base" type="fixed">
@@ -38,39 +38,39 @@
         </link>
         <!-- virtual links for convex shapes of chair parts -->
-        <link name="${prefix}back_support"/>
-        <joint name="${prefix}back_joint" type="fixed">
-            <parent link="${prefix}main"/>
-            <child link="${prefix}back_support"/>
-        </joint>
-        <link name="${prefix}left_handle"/>
-        <joint name="${prefix}lhandle_joint" type="fixed">
-            <parent link="${prefix}main"/>
-            <child link="${prefix}left_handle"/>
-        </joint>
-        <link name="${prefix}right_handle"/>
-        <joint name="${prefix}rhandle_joint" type="fixed">
-            <parent link="${prefix}main"/>
-            <child link="${prefix}right_handle"/>
-        </joint>
-        <link name="${prefix}leg_fl"/>
-        <joint name="${prefix}leg_fl_joint" type="fixed">
-            <parent link="${prefix}main"/>
-            <child link="${prefix}leg_fl"/>
-        </joint>
-        <link name="${prefix}leg_fr"/>
-        <joint name="${prefix}leg_fr_joint" type="fixed">
-            <parent link="${prefix}main"/>
-            <child link="${prefix}leg_fr"/>
-        </joint>
-        <link name="${prefix}leg_rl"/>
-        <joint name="${prefix}leg_rl_joint" type="fixed">
-            <parent link="${prefix}main"/>
-            <child link="${prefix}leg_rl"/>
-        </joint>
-        <link name="${prefix}leg_rr"/>
-        <joint name="${prefix}leg_rr_joint" type="fixed">
-            <parent link="${prefix}main"/>
-            <child link="${prefix}leg_rr"/>
-        </joint>
+<!--        <link name="${prefix}back_support"/>-->
+<!--        <joint name="${prefix}back_joint" type="fixed">-->
+<!--            <parent link="${prefix}main"/>-->
+<!--            <child link="${prefix}back_support"/>-->
+<!--        </joint>-->
+<!--        <link name="${prefix}left_handle"/>-->
+<!--        <joint name="${prefix}lhandle_joint" type="fixed">-->
+<!--            <parent link="${prefix}main"/>-->
+<!--            <child link="${prefix}left_handle"/>-->
+<!--        </joint>-->
+<!--        <link name="${prefix}right_handle"/>-->
+<!--        <joint name="${prefix}rhandle_joint" type="fixed">-->
+<!--            <parent link="${prefix}main"/>-->
+<!--            <child link="${prefix}right_handle"/>-->
+<!--        </joint>-->
+<!--        <link name="${prefix}leg_fl"/>-->
+<!--        <joint name="${prefix}leg_fl_joint" type="fixed">-->
+<!--            <parent link="${prefix}main"/>-->
+<!--            <child link="${prefix}leg_fl"/>-->
+<!--        </joint>-->
+<!--        <link name="${prefix}leg_fr"/>-->
+<!--        <joint name="${prefix}leg_fr_joint" type="fixed">-->
+<!--            <parent link="${prefix}main"/>-->
+<!--            <child link="${prefix}leg_fr"/>-->
+<!--        </joint>-->
+<!--        <link name="${prefix}leg_rl"/>-->
+<!--        <joint name="${prefix}leg_rl_joint" type="fixed">-->
+<!--            <parent link="${prefix}main"/>-->
+<!--            <child link="${prefix}leg_rl"/>-->
+<!--        </joint>-->
+<!--        <link name="${prefix}leg_rr"/>-->
+<!--        <joint name="${prefix}leg_rr_joint" type="fixed">-->
+<!--            <parent link="${prefix}main"/>-->
+<!--            <child link="${prefix}leg_rr"/>-->
+<!--        </joint>-->
     </xacro:macro>
 </robot>

File: objects_descriptions/urdf/qolo.xacro (robot description, xacro)
@@ -9,20 +9,20 @@
             <color rgba="0.4 0.4 0.4 1"/>
         </material>
-        <xacro:if value="${connected_to == ''}">
-            <link name="world"/>
-            <xacro:property name="base_frame_name" value="world"/>
-        </xacro:if>
-        <xacro:unless value="${connected_to == ''}">
-            <xacro:property name="base_frame_name" value="${connected_to}"/>
-        </xacro:unless>
-        <xacro:if value="${connected_to == 'odom'}">
-            <link name="odom"/>
-            <xacro:property name="base_frame_name" value="odom"/>
-        </xacro:if>
-        <joint name="${prefix}base_to_${base_frame_name}" type="fixed">
-            <parent link="${base_frame_name}"/>
-            <child link="${prefix}tf"/>
-            <origin rpy="${rpy}" xyz="${xyz}"/>
-        </joint>
+<!--        <xacro:if value="${connected_to == ''}">-->
+<!--            <link name="world"/>-->
+<!--            <xacro:property name="base_frame_name" value="world"/>-->
+<!--        </xacro:if>-->
+<!--        <xacro:unless value="${connected_to == ''}">-->
+<!--            <xacro:property name="base_frame_name" value="${connected_to}"/>-->
+<!--        </xacro:unless>-->
+<!--        <xacro:if value="${connected_to == 'odom'}">-->
+<!--            <link name="odom"/>-->
+<!--            <xacro:property name="base_frame_name" value="odom"/>-->
+<!--        </xacro:if>-->
+<!--        <joint name="${prefix}base_to_${base_frame_name}" type="fixed">-->
+<!--            <parent link="${base_frame_name}"/>-->
+<!--            <child link="${prefix}tf"/>-->
+<!--            <origin rpy="${rpy}" xyz="${xyz}"/>-->
+<!--        </joint>-->
         <link name="${prefix}tf">
             <inertial>

Commit message: Added scenarios for controller evaluation

File: objects_descriptions/urdf/chair.xacro (robot description, xacro)
@@ -38,39 +38,39 @@
         </link>
         <!-- virtual links for convex shapes of chair parts -->
-<!--        <link name="${prefix}back_support"/>-->
-<!--        <joint name="${prefix}back_joint" type="fixed">-->
-<!--            <parent link="${prefix}main"/>-->
-<!--            <child link="${prefix}back_support"/>-->
-<!--        </joint>-->
-<!--        <link name="${prefix}left_handle"/>-->
-<!--        <joint name="${prefix}lhandle_joint" type="fixed">-->
-<!--            <parent link="${prefix}main"/>-->
-<!--            <child link="${prefix}left_handle"/>-->
-<!--        </joint>-->
-<!--        <link name="${prefix}right_handle"/>-->
-<!--        <joint name="${prefix}rhandle_joint" type="fixed">-->
-<!--            <parent link="${prefix}main"/>-->
-<!--            <child link="${prefix}right_handle"/>-->
-<!--        </joint>-->
-<!--        <link name="${prefix}leg_fl"/>-->
-<!--        <joint name="${prefix}leg_fl_joint" type="fixed">-->
-<!--            <parent link="${prefix}main"/>-->
-<!--            <child link="${prefix}leg_fl"/>-->
-<!--        </joint>-->
-<!--        <link name="${prefix}leg_fr"/>-->
-<!--        <joint name="${prefix}leg_fr_joint" type="fixed">-->
-<!--            <parent link="${prefix}main"/>-->
-<!--            <child link="${prefix}leg_fr"/>-->
-<!--        </joint>-->
-<!--        <link name="${prefix}leg_rl"/>-->
-<!--        <joint name="${prefix}leg_rl_joint" type="fixed">-->
-<!--            <parent link="${prefix}main"/>-->
-<!--            <child link="${prefix}leg_rl"/>-->
-<!--        </joint>-->
-<!--        <link name="${prefix}leg_rr"/>-->
-<!--        <joint name="${prefix}leg_rr_joint" type="fixed">-->
-<!--            <parent link="${prefix}main"/>-->
-<!--            <child link="${prefix}leg_rr"/>-->
-<!--        </joint>-->
+        <link name="${prefix}back_support"/>
+        <joint name="${prefix}back_joint" type="fixed">
+            <parent link="${prefix}main"/>
+            <child link="${prefix}back_support"/>
+        </joint>
+        <link name="${prefix}left_handle"/>
+        <joint name="${prefix}lhandle_joint" type="fixed">
+            <parent link="${prefix}main"/>
+            <child link="${prefix}left_handle"/>
+        </joint>
+        <link name="${prefix}right_handle"/>
+        <joint name="${prefix}rhandle_joint" type="fixed">
+            <parent link="${prefix}main"/>
+            <child link="${prefix}right_handle"/>
+        </joint>
+        <link name="${prefix}leg_fl"/>
+        <joint name="${prefix}leg_fl_joint" type="fixed">
+            <parent link="${prefix}main"/>
+            <child link="${prefix}leg_fl"/>
+        </joint>
+        <link name="${prefix}leg_fr"/>
+        <joint name="${prefix}leg_fr_joint" type="fixed">
+            <parent link="${prefix}main"/>
+            <child link="${prefix}leg_fr"/>
+        </joint>
+        <link name="${prefix}leg_rl"/>
+        <joint name="${prefix}leg_rl_joint" type="fixed">
+            <parent link="${prefix}main"/>
+            <child link="${prefix}leg_rl"/>
+        </joint>
+        <link name="${prefix}leg_rr"/>
+        <joint name="${prefix}leg_rr_joint" type="fixed">
+            <parent link="${prefix}main"/>
+            <child link="${prefix}leg_rr"/>
+        </joint>
     </xacro:macro>
 </robot>
