Commit message: Updated launch files to fix multiple robots with the same frame. Added a launch file to connect the DSM to Rviz (broken)

File: objects_descriptions/urdf/table.xacro (robot description, xacro)
@@ -19,8 +19,8 @@
 <!--        <joint name="${prefix}base_to_${base_frame_name}" type="fixed">-->
 <!--            <parent link="${base_frame_name}"/>-->
-<!--            <child link="${prefix}main_link"/>-->
+<!--            <child link="${prefix}base_link"/>-->
 <!--            <origin rpy="${rpy}" xyz="${xyz}"/>-->
 <!--        </joint>-->
-        <link name="${prefix}main_link">
+        <link name="${prefix}base_link">
             <visual>
                 <geometry>
