Commit message: updated urdf model to include a fixed parameter

File: objects_descriptions/urdf/chair.urdf.xacro (robot description, xacro)
@@ -6,6 +6,7 @@
     <xacro:arg name="rpy" default="'0 0 0'"/>
     <xacro:arg name="mass" default="2.0"/>
+    <xacro:arg name="fixed" default="1"/>
     <xacro:include filename="$(find objects_descriptions)/urdf/chair.xacro"/>
     <xacro:chair prefix="$(arg prefix)" connected_to="$(arg connected_to)" xyz="$(arg xyz)" rpy="$(arg rpy)"
-                 mass="$(arg mass)"/>
+                 mass="$(arg mass)" fixed="$(arg fixed)"/>
 </robot>

File: objects_descriptions/urdf/chair.xacro (robot description, xacro)
@@ -2,21 +2,23 @@
 <robot name="chair_sim" xmlns:xacro="http://wiki.ros.org/xacro">
     <xacro:macro name="chair"
-                 params="prefix='chair_' connected_to:='' xyz:='0 0 0' rpy:='0 0 0' mass=2.0">
-<!--        <xacro:if value="${connected_to == ''}">-->
-<!--            <link name="world"/>-->
-<!--            <xacro:property name="base_frame_name" value="world"/>-->
-<!--        </xacro:if>-->
-<!--        <xacro:unless value="${connected_to == ''}">-->
-<!--            <xacro:property name="base_frame_name" value="${connected_to}"/>-->
-<!--        </xacro:unless>-->
-<!--        <xacro:if value="${connected_to == 'odom'}">-->
-<!--            <link name="odom"/>-->
-<!--            <xacro:property name="base_frame_name" value="odom"/>-->
-<!--        </xacro:if>-->
-<!--        <joint name="${prefix}base_to_${base_frame_name}" type="fixed">-->
-<!--            <parent link="${base_frame_name}"/>-->
-<!--            <child link="${prefix}base_link"/>-->
-<!--            <origin rpy="${rpy}" xyz="${xyz}"/>-->
-<!--        </joint>-->
+                 params="prefix='chair_' connected_to:='' xyz:='0 0 0' rpy:='0 0 0' mass=2.0, fixed:=1">
+        <xacro:if value="${fixed == 1}">
+            <xacro:if value="${connected_to == ''}">
+                <link name="world"/>
+                <xacro:property name="base_frame_name" value="world"/>
+            </xacro:if>
+            <xacro:unless value="${connected_to == ''}">
+                <xacro:property name="base_frame_name" value="${connected_to}"/>
+            </xacro:unless>
+            <xacro:if value="${connected_to == 'odom'}">
+                <link name="odom"/>
+                <xacro:property name="base_frame_name" value="odom"/>
+            </xacro:if>
+            <joint name="${prefix}base_to_${base_frame_name}" type="fixed">
+                <parent link="${base_frame_name}"/>
+                <child link="${prefix}base_link"/>
+                <origin rpy="${rpy}" xyz="${xyz}"/>
+            </joint>
+        </xacro:if>
         <link name="${prefix}base_link"/>
         <joint name="${prefix}base" type="fixed">

File: objects_descriptions/urdf/qolo.urdf.xacro (robot description, xacro)
@@ -6,6 +6,7 @@
     <xacro:arg name="rpy" default="'0 0 0'"/>
     <xacro:arg name="mass" default="3.0"/>
+    <xacro:arg name="fixed" default="1"/>
     <xacro:include filename="$(find objects_descriptions)/urdf/qolo.xacro"/>
     <xacro:qolo prefix="$(arg prefix)" connected_to="$(arg connected_to)" xyz="$(arg xyz)" rpy="$(arg rpy)"
-                 mass="$(arg mass)"/>
+                 mass="$(arg mass)" fixed="$(arg fixed)"/>
 </robot>

File: objects_descriptions/urdf/qolo.xacro (robot description, xacro)
@@ -2,5 +2,5 @@
 <robot name="qolo_sim" xmlns:xacro="http://wiki.ros.org/xacro">
     <xacro:macro name="qolo"
-                 params="prefix='qolo_' connected_to:='' xyz:='0 0 0' rpy:='0 0 0' mass=3.0">
+                 params="prefix='qolo_' connected_to:='' xyz:='0 0 0' rpy:='0 0 0' mass=3.0, fixed:=1">
         <material name="gray">
             <color rgba="0.7 0.7 0.7 1"/>
@@ -9,20 +9,22 @@
             <color rgba="0.4 0.4 0.4 1"/>
         </material>
-<!--        <xacro:if value="${connected_to == ''}">-->
-<!--            <link name="world"/>-->
-<!--            <xacro:property name="base_frame_name" value="world"/>-->
-<!--        </xacro:if>-->
-<!--        <xacro:unless value="${connected_to == ''}">-->
-<!--            <xacro:property name="base_frame_name" value="${connected_to}"/>-->
-<!--        </xacro:unless>-->
-<!--        <xacro:if value="${connected_to == 'odom'}">-->
-<!--            <link name="odom"/>-->
-<!--            <xacro:property name="base_frame_name" value="odom"/>-->
-<!--        </xacro:if>-->
-<!--        <joint name="${prefix}base_to_${base_frame_name}" type="fixed">-->
-<!--            <parent link="${base_frame_name}"/>-->
-<!--            <child link="${prefix}base_link"/>-->
-<!--            <origin rpy="${rpy}" xyz="${xyz}"/>-->
-<!--        </joint>-->
+        <xacro:if value="${fixed == 1}">
+            <xacro:if value="${connected_to == ''}">
+                <link name="world"/>
+                <xacro:property name="base_frame_name" value="world"/>
+            </xacro:if>
+            <xacro:unless value="${connected_to == ''}">
+                <xacro:property name="base_frame_name" value="${connected_to}"/>
+            </xacro:unless>
+            <xacro:if value="${connected_to == 'odom'}">
+                <link name="odom"/>
+                <xacro:property name="base_frame_name" value="odom"/>
+            </xacro:if>
+            <joint name="${prefix}base_to_${base_frame_name}" type="fixed">
+                <parent link="${base_frame_name}"/>
+                <child link="${prefix}base_link"/>
+                <origin rpy="${rpy}" xyz="${xyz}"/>
+            </joint>
+        </xacro:if>
         <link name="${prefix}base_link">
             <inertial>

File: objects_descriptions/urdf/table.urdf.xacro (robot description, xacro)
@@ -6,6 +6,7 @@
     <xacro:arg name="rpy" default="'0 0 0'"/>
     <xacro:arg name="mass" default="8.0"/>
+    <xacro:arg name="fixed" default="1"/>
     <xacro:include filename="$(find objects_descriptions)/urdf/table.xacro"/>
     <xacro:table prefix="$(arg prefix)" connected_to="$(arg connected_to)" xyz="$(arg xyz)" rpy="$(arg rpy)"
-                 mass="$(arg mass)"/>
+                 mass="$(arg mass)" fixed="$(arg fixed)"/>
 </robot>

File: objects_descriptions/urdf/table.xacro (robot description, xacro)
@@ -2,24 +2,26 @@
 <robot name="table_sim" xmlns:xacro="http://wiki.ros.org/xacro">
     <xacro:macro name="table"
-                 params="prefix='table_' connected_to:='' xyz:='0 0 0' rpy:='0 0 0' mass=3.0">
+                 params="prefix='table_' connected_to:='' xyz:='0 0 0' rpy:='0 0 0' mass=3.0, fixed:=1">
         <material name="Shape.003">
             <color rgba="0.33 0.24 0.15 1"/>
         </material>
-<!--        <xacro:if value="${connected_to == ''}">-->
-<!--            <link name="world"/>-->
-<!--            <xacro:property name="base_frame_name" value="world"/>-->
-<!--        </xacro:if>-->
-<!--        <xacro:unless value="${connected_to == ''}">-->
-<!--            <xacro:property name="base_frame_name" value="${connected_to}"/>-->
-<!--        </xacro:unless>-->
-<!--        <xacro:if value="${connected_to == 'odom'}">-->
-<!--            <link name="odom"/>-->
-<!--            <xacro:property name="base_frame_name" value="odom"/>-->
-<!--        </xacro:if>-->
-<!--        <joint name="${prefix}base_to_${base_frame_name}" type="fixed">-->
-<!--            <parent link="${base_frame_name}"/>-->
-<!--            <child link="${prefix}base_link"/>-->
-<!--            <origin rpy="${rpy}" xyz="${xyz}"/>-->
-<!--        </joint>-->
+        <xacro:if value="${fixed == 1}">
+            <xacro:if value="${connected_to == ''}">
+                <link name="world"/>
+                <xacro:property name="base_frame_name" value="world"/>
+            </xacro:if>
+            <xacro:unless value="${connected_to == ''}">
+                <xacro:property name="base_frame_name" value="${connected_to}"/>
+            </xacro:unless>
+            <xacro:if value="${connected_to == 'odom'}">
+                <link name="odom"/>
+                <xacro:property name="base_frame_name" value="odom"/>
+            </xacro:if>
+            <joint name="${prefix}base_to_${base_frame_name}" type="fixed">
+                <parent link="${base_frame_name}"/>
+                <child link="${prefix}base_link"/>
+                <origin rpy="${rpy}" xyz="${xyz}"/>
+            </joint>
+        </xacro:if>
         <link name="${prefix}base_link">
             <visual>

File: objects_descriptions/urdf/wheelchair.urdf.xacro (robot description, xacro)
@@ -1,11 +1,12 @@
 <?xml version="1.0"?>
 <robot name="wheelchair" xmlns:xacro="http://wiki.ros.org/xacro">
-    <xacro:arg name="prefix" default="wheelchair"/>
+    <xacro:arg name="prefix" default="wheelchair_"/>
     <xacro:arg name="connected_to" default=""/>
     <xacro:arg name="xyz" default="'0 0 0'"/>
     <xacro:arg name="rpy" default="'0 0 0'"/>
     <xacro:arg name="mass" default="3.0"/>
+    <xacro:arg name="fixed" default="1"/>
     <xacro:include filename="$(find objects_descriptions)/urdf/wheelchair.xacro"/>
     <xacro:wheelchair prefix="$(arg prefix)" connected_to="$(arg connected_to)" xyz="$(arg xyz)" rpy="$(arg rpy)"
-                      mass="$(arg mass)"/>
+                      mass="$(arg mass)" fixed="$(arg fixed)"/>
 </robot>

File: objects_descriptions/urdf/wheelchair.xacro (robot description, xacro)
@@ -2,21 +2,23 @@
 <robot name="wheelchair_sim" xmlns:xacro="http://wiki.ros.org/xacro">
     <xacro:macro name="wheelchair"
-                 params="prefix='wheelchair_' connected_to:='' xyz:='0 0 0' rpy:='0 0 0' mass=3.0">
-        <xacro:if value="${connected_to == ''}">
-            <link name="world"/>
-            <xacro:property name="base_frame_name" value="world"/>
+                 params="prefix='wheelchair_' connected_to:='' xyz:='0 0 0' rpy:='0 0 0' mass=3.0, fixed:=1">
+        <xacro:if value="${fixed == 1}">
+            <xacro:if value="${connected_to == ''}">
+                <link name="world"/>
+                <xacro:property name="base_frame_name" value="world"/>
+            </xacro:if>
+            <xacro:unless value="${connected_to == ''}">
+                <xacro:property name="base_frame_name" value="${connected_to}"/>
+            </xacro:unless>
+            <xacro:if value="${connected_to == 'odom'}">
+                <link name="odom"/>
+                <xacro:property name="base_frame_name" value="odom"/>
+            </xacro:if>
+            <joint name="${prefix}base_to_${base_frame_name}" type="fixed">
+                <parent link="${base_frame_name}"/>
+                <child link="${prefix}base_link"/>
+                <origin rpy="${rpy}" xyz="${xyz}"/>
+            </joint>
         </xacro:if>
-        <xacro:unless value="${connected_to == ''}">
-            <xacro:property name="base_frame_name" value="${connected_to}"/>
-        </xacro:unless>
-        <xacro:if value="${connected_to == 'odom'}">
-            <link name="odom"/>
-            <xacro:property name="base_frame_name" value="odom"/>
-        </xacro:if>
-        <joint name="${prefix}base_to_${base_frame_name}" type="fixed">
-            <parent link="${base_frame_name}"/>
-            <child link="${prefix}base_link"/>
-            <origin rpy="${rpy}" xyz="${xyz}"/>
-        </joint>
         <link name="${prefix}base_link"/>
         <joint name="${prefix}base" type="fixed">
