Commit message: updated DSM code for Rviz

File: objects_descriptions/urdf/hospital_bed.xacro (robot description, xacro)
@@ -33,7 +33,7 @@
             </visual>
             <collision>
-<!--                <origin xyz="0 0 0" rpy="0 0 0"/>-->
+                <origin xyz="0 0.45 0" rpy="0 0 0"/>
                 <geometry>
-                    <box size="2 0.9 0.5"/>
+                    <box size="2.2 0.9 1.1"/>
                 </geometry>
             </collision>
