Commit message: fixed the DSM visualisation with Rviz

File: objects_descriptions/urdf/qolo.xacro (robot description, xacro)
@@ -22,8 +22,8 @@
 <!--        <joint name="${prefix}base_to_${base_frame_name}" type="fixed">-->
 <!--            <parent link="${base_frame_name}"/>-->
-<!--            <child link="${prefix}tf"/>-->
+<!--            <child link="${prefix}base_link"/>-->
 <!--            <origin rpy="${rpy}" xyz="${xyz}"/>-->
 <!--        </joint>-->
-        <link name="${prefix}tf">
+        <link name="${prefix}base_link">
             <inertial>
                 <origin rpy="0 0 0" xyz="-0.160 0 0.184"/>
@@ -67,5 +67,5 @@
         </link>
         <joint name="${prefix}main_to_wheel_right" type="fixed">
-            <parent link="${prefix}tf"/>
+            <parent link="${prefix}base_link"/>
             <child link="${prefix}wheel_right"/>
             <origin xyz="0 0.2 0"/>
@@ -93,5 +93,5 @@
         </link>
         <joint name="${prefix}main_to_wheel_left" type="fixed">
-            <parent link="${prefix}tf"/>
+            <parent link="${prefix}base_link"/>
             <child link="${prefix}wheel_left"/>
             <origin xyz="0 -0.2 0"/>
@@ -120,5 +120,5 @@
         </link>
         <joint name="${prefix}main_to_bumper" type="fixed">
-            <parent link="${prefix}tf"/>
+            <parent link="${prefix}base_link"/>
             <child link="${prefix}bumper"/>
             <origin xyz="0.035 0 0.015"/>

Commit message: Human model added into Qolo URDF

File: objects_descriptions/urdf/qolo.xacro (robot description, xacro)
@@ -127,4 +127,804 @@
             <axis xyz="1 0 0"/>
         </joint>
+        <joint name="base" type="fixed">
+	    <parent link="${prefix}base_link"/>
+	    <child link="HipsLink"/>
+	    <origin rpy="0 0 0" xyz="-0.25 0 0.87"/>
+	 </joint>
+        <link name="HipsLink">
+	    <inertial>
+	      <origin rpy="0 0 0" xyz="-0.0232 0.0 -0.1192"/>
+	      <mass value="20.9238"/>
+	      <inertia ixx="-0.3225" ixy="-0.0" ixz="-0.0" iyy="0.0" iyz="0.2362" izz="0.0"/>
+	    </inertial>
+	    <visual>
+	      <origin rpy="0 0 0" xyz="0 0 0"/>
+	      <geometry>
+		<mesh filename="package://objects_descriptions/meshes/human/HipsLinkFull.dae"/>
+	      </geometry>
+	    </visual>
+	    <collision>
+	      <origin rpy="0 0 0" xyz="0 0 0"/>
+	      <geometry>
+		<mesh filename="package://objects_descriptions/meshes/human/HipsLinkFull.dae"/>
+	      </geometry>
+	    </collision>
+	 </link>
+	 <link name="TorsoLink">
+	    <inertial>
+	      <origin rpy="0 0 0" xyz="-0.1334 0.0 0.4701"/>
+	      <mass value="10.7790"/>
+	      <inertia ixx="-0.3481" ixy="-0.0" ixz="-0.0" iyy="0.0" iyz="0.2709" izz="0.0"/>
+	    </inertial>
+	    <visual>
+	      <origin rpy="0 0 0" xyz="0 0 0"/>
+	      <geometry>
+		<mesh filename="package://objects_descriptions/meshes/human/TorsoLinkFull.dae"/>
+	      </geometry>
+	    </visual>
+	    <collision>
+	      <origin rpy="0 0 0" xyz="0 0 0"/>
+	      <geometry>
+		<mesh filename="package://objects_descriptions/meshes/human/TorsoLinkFull.dae"/>
+	      </geometry>
+	    </collision>
+	 </link>
+	 <link name="HeadLink">
+	    <inertial>
+	      <origin rpy="0 0 0" xyz="0.0459 0.0 0.0433"/>
+	      <mass value="4.7372"/>
+	      <inertia ixx="-0.1891" ixy="-0.0" ixz="-0.0" iyy="0.0" iyz="0.1891" izz="0.0"/>
+	    </inertial>
+	    <visual>
+	      <origin rpy="0 0 0" xyz="0 0 0"/>
+	      <geometry>
+		<mesh filename="package://objects_descriptions/meshes/human/HeadLinkFull.dae"/>
+	      </geometry>
+	    </visual>
+	    <collision>
+	      <origin rpy="0 0 0" xyz="0 0 0"/>
+	      <geometry>
+		<mesh filename="package://objects_descriptions/meshes/human/HeadLinkFull.dae"/>
+	      </geometry>
+	    </collision>
+	 </link>
+	 <link name="LLegLink">
+	    <inertial>
+	      <origin rpy="0 0 0" xyz="-0.0185 -0.0071 -0.178"/>
+	      <mass value="6.51"/>
+	      <inertia ixx="-0.1264" ixy="-0.0" ixz="-0.0" iyy="0.0" iyz="0.1264" izz="0.0"/>
+	    </inertial>
+	    <visual>
+	      <origin rpy="0 0 0" xyz="0 0 0"/>
+	      <geometry>
+		<mesh filename="package://objects_descriptions/meshes/human/LLegLink.dae"/>
+	      </geometry>
+	    </visual>
+	    <collision>
+	      <origin rpy="0 0 0" xyz="0 0 0"/>
+	      <geometry>
+		<mesh filename="package://objects_descriptions/meshes/human/LLegLink.dae"/>
+	      </geometry>
+	    </collision>
+	  </link>
+	  <link name="LShinLink">
+	    <inertial>
+	      <origin rpy="0 0 0" xyz="-0.0131 0.0025 0.0346"/>
+	      <mass value="3.095"/>
+	      <inertia ixx="-0.0632" ixy="-0.0" ixz="-0.0" iyy="0.0" iyz="0.0632" izz="0.0"/>
+	    </inertial>
+	    <visual>
+	      <origin rpy="0 0 0" xyz="0 0 0"/>
+	      <geometry>
+		<mesh filename="package://objects_descriptions/meshes/human/LShinLink.dae"/>
+	      </geometry>
+	    </visual>
+	    <collision>
+	      <origin rpy="0 0 0" xyz="0 0 0"/>
+	      <geometry>
+		<mesh filename="package://objects_descriptions/meshes/human/LShinLink.dae"/>
+	      </geometry>
+	    </collision>
+	  </link>
+	  <link name="LAnkleLink">
+	    <inertial>
+	      <origin rpy="0 0 0" xyz="0.0508 0.0067 -0.0646"/>
+	      <mass value="0.99"/>
+	      <inertia ixx="-0.0015" ixy="-0.0" ixz="-0.0" iyy="0.0" iyz="0.0059" izz="0.0"/>
+	    </inertial>
+	    <visual>
+	      <origin rpy="0 0 0" xyz="0 0 0"/>
+	      <geometry>
+		<mesh filename="package://objects_descriptions/meshes/human/LAnkleLinkFull.dae"/>
+	      </geometry>
+	    </visual>
+	    <collision>
+	      <origin rpy="0 0 0" xyz="0 0 0"/>
+	      <geometry>
+		<mesh filename="package://objects_descriptions/meshes/human/LAnkleLinkFull.dae"/>
+	      </geometry>
+	    </collision>
+	  </link>
+	  <link name="RLegLink">
+	    <inertial>
+	      <origin rpy="0 0 0" xyz="-0.0185 -0.0071 -0.178"/>
+	      <mass value="6.51"/>
+	      <inertia ixx="-0.1264" ixy="-0.0" ixz="-0.0" iyy="0.0" iyz="0.1264" izz="0.0"/>
+	    </inertial>
+	    <visual>
+	      <origin rpy="0 0 0" xyz="0 0 0"/>
+	      <geometry>
+		<mesh filename="package://objects_descriptions/meshes/human/RLegLink.dae"/>
+	      </geometry>
+	    </visual>
+	    <collision>
+	      <origin rpy="0 0 0" xyz="0 0 0"/>
+	      <geometry>
+		<mesh filename="package://objects_descriptions/meshes/human/RLegLink.dae"/>
+	      </geometry>
+	    </collision>
+	  </link>
+	  <link name="RShinLink">
+	    <inertial>
+	      <origin rpy="0 0 0" xyz="-0.0131 0.0025 0.0346"/>
+	      <mass value="3.095"/>
+	      <inertia ixx="-0.0632" ixy="-0.0" ixz="-0.0" iyy="0.0" iyz="0.0632" izz="0.0"/>
+	    </inertial>
+	    <visual>
+	      <origin rpy="0 0 0" xyz="0 0 0"/>
+	      <geometry>
+		<mesh filename="package://objects_descriptions/meshes/human/RShinLink.dae"/>
+	      </geometry>
+	    </visual>
+	    <collision>
+	      <origin rpy="0 0 0" xyz="0 0 0"/>
+	      <geometry>
+		<mesh filename="package://objects_descriptions/meshes/human/RShinLink.dae"/>
+	      </geometry>
+	    </collision>
+	  </link>
+	  <link name="RAnkleLink">
+	    <inertial>
+	      <origin rpy="0 0 0" xyz="0.0508 -0.0067 -0.0646"/>
+	      <mass value="0.99"/>
+	      <inertia ixx="-0.0015" ixy="-0.0" ixz="-0.0" iyy="0.0" iyz="0.0059" izz="0.0"/>
+	    </inertial>
+	    <visual>
+	      <origin rpy="0 0 0" xyz="0 0 0"/>
+	      <geometry>
+		<mesh filename="package://objects_descriptions/meshes/human/RAnkleLinkFull.dae"/>
+	      </geometry>
+	    </visual>
+	    <collision>
+	      <origin rpy="0 0 0" xyz="0 0 0"/>
+	      <geometry>
+		<mesh filename="package://objects_descriptions/meshes/human/RAnkleLinkFull.dae"/>
+	      </geometry>
+	    </collision>
+	  </link>
+	    <link name="LArmLink">
+	    <inertial>
+	      <origin rpy="0 0 0" xyz="-0.0 0.1328 0.0"/>
+	      <mass value="1.96"/>
+	      <inertia ixx="-0.3475" ixy="-0.0" ixz="-0.0" iyy="0.0" iyz="0.6719" izz="0.0"/>
+	    </inertial>
+	    <visual>
+	      <origin rpy="0 0 0" xyz="0 0 0"/>
+	      <geometry>
+		<mesh filename="package://objects_descriptions/meshes/human/LArmLinkFull.dae"/>
+	      </geometry>
+	    </visual>
+	    <collision>
+	      <origin rpy="0 0 0" xyz="0 0 0"/>
+	      <geometry>
+		<mesh filename="package://objects_descriptions/meshes/human/LArmLinkFull.dae"/>
+	      </geometry>
+	    </collision>
+	  </link>
+	  <link name="LElbowLink">
+	    <inertial>
+	      <origin rpy="0 0 0" xyz="0.000513 0.034528 -0.000934"/>
+	      <mass value="0.25"/>
+	      <inertia ixx="-5.9e-05" ixy="-0.0" ixz="-0.0" iyy="0.0" iyz="8e-05" izz="0.0"/>
+	    </inertial>
+	    <visual>
+	      <origin rpy="0 0 0" xyz="0 0 0"/>
+	      <geometry>
+		<mesh filename="package://objects_descriptions/meshes/human/LElbowLink.dae"/>
+	      </geometry>
+	    </visual>
+	    <collision>
+	      <origin rpy="0 0 0" xyz="0 0 0"/>
+	      <geometry>
+		<mesh filename="package://objects_descriptions/meshes/human/LElbowLink.dae"/>
+	      </geometry>
+	    </collision>
+	  </link>
+	  <link name="LForearmLink">
+	    <inertial>
+	      <origin rpy="0 0 0" xyz="-0.0 0.15114 0.0"/>
+	      <mass value="1.18"/>
+	      <inertia ixx="-0.0753" ixy="-0.0" ixz="-0.0" iyy="0.0" iyz="0.1326" izz="0.0"/>
+	    </inertial>
+	    <visual>
+	      <origin rpy="0 0 0" xyz="0 0 0"/>
+	      <geometry>
+		<mesh filename="package://objects_descriptions/meshes/human/LForearmLink.dae"/>
+	      </geometry>
+	    </visual>
+	    <collision>
+	      <origin rpy="0 0 0" xyz="0 0 0"/>
+	      <geometry>
+		<mesh filename="package://objects_descriptions/meshes/human/LForearmLink.dae"/>
+	      </geometry>
+	    </collision>
+	  </link>
+	  <link name="LHandLink">
+	    <inertial>
+	      <origin rpy="0 0 0" xyz="0.0139 0.042 -0.0128"/>
+	      <mass value="0.272"/>
+	      <inertia ixx="-0.00029946" ixy="-0.0" ixz="-0.0" iyy="0.0" iyz="0.00019118" izz="0.0"/>
+	    </inertial>
+	    <visual>
+	      <origin rpy="0 0 0" xyz="0 0 0"/>
+	      <geometry>
+		<mesh filename="package://objects_descriptions/meshes/human/LWrist.dae"/>
+	      </geometry>
+	    </visual>
+	    <collision>
+	      <origin rpy="0 0 0" xyz="0 0 0"/>
+	      <geometry>
+		<mesh filename="package://objects_descriptions/meshes/human/LWrist.dae"/>
+	      </geometry>
+	    </collision>
+	  </link>
+	  <link name="RArmLink">
+	    <inertial>
+	      <origin rpy="0 0 0" xyz="-0.0 -0.1328 0.0"/>
+	      <mass value="1.96"/>
+	      <inertia ixx="-0.3475" ixy="-0.0" ixz="-0.0" iyy="0.0" iyz="0.6719" izz="0.0"/>
+	    </inertial>
+	    <visual>
+	      <origin rpy="0 0 0" xyz="0 0 0"/>
+	      <geometry>
+		<mesh filename="package://objects_descriptions/meshes/human/RArmLinkFull.dae"/>
+	      </geometry>
+	    </visual>
+	    <collision>
+	      <origin rpy="0 0 0" xyz="0 0 0"/>
+	      <geometry>
+		<mesh filename="package://objects_descriptions/meshes/human/RArmLinkFull.dae"/>
+	      </geometry>
+	    </collision>
+	  </link>
+	  <link name="RElbowLink">
+	    <inertial>
+	      <origin rpy="0 0 0" xyz="0.000513 -0.034528 -0.000934"/>
+	      <mass value="0.25"/>
+	      <inertia ixx="-5.9e-05" ixy="-0.0" ixz="-0.0" iyy="0.0" iyz="8e-05" izz="0.0"/>
+	    </inertial>
+	    <visual>
+	      <origin rpy="0 0 0" xyz="0 0 0"/>
+	      <geometry>
+		<mesh filename="package://objects_descriptions/meshes/human/RElbowLink.dae"/>
+	      </geometry>
+	    </visual>
+	    <collision>
+	      <origin rpy="0 0 0" xyz="0 0 0"/>
+	      <geometry>
+		<mesh filename="package://objects_descriptions/meshes/human/RElbowLink.dae"/>
+	      </geometry>
+	    </collision>
+	  </link>
+	  <link name="RForearmLink">
+	    <inertial>
+	      <origin rpy="0 0 0" xyz="-0.0 -0.15114 0.0"/>
+	      <mass value="1.18"/>
+	      <inertia ixx="-0.0753" ixy="-0.0" ixz="-0.0" iyy="0.0" iyz="0.1326" izz="0.0"/>
+	    </inertial>
+	    <visual>
+	      <origin rpy="0 0 0" xyz="0 0 0"/>
+	      <geometry>
+		<mesh filename="package://objects_descriptions/meshes/human/RForearmLink.dae"/>
+	      </geometry>
+	    </visual>
+	    <collision>
+	      <origin rpy="0 0 0" xyz="0 0 0"/>
+	      <geometry>
+		<mesh filename="package://objects_descriptions/meshes/human/RForearmLink.dae"/>
+	      </geometry>
+	    </collision>
+	  </link>
+	  <link name="RHandLink">
+	    <inertial>
+	      <origin rpy="0 0 0" xyz="0.0139 -0.042 -0.0128"/>
+	      <mass value="0.272"/>
+	      <inertia ixx="-0.00029946" ixy="-0.0" ixz="-0.0" iyy="0.0" iyz="0.00019118" izz="0.0"/>
+	    </inertial>
+	    <visual>
+	      <origin rpy="0 0 0" xyz="0 0 0"/>
+	      <geometry>
+		<mesh filename="package://objects_descriptions/meshes/human/RWrist.dae"/>
+	      </geometry>
+	    </visual>
+	    <collision>
+	      <origin rpy="0 0 0" xyz="0 0 0"/>
+	      <geometry>
+		<mesh filename="package://objects_descriptions/meshes/human/RWrist.dae"/>
+	      </geometry>
+	    </collision>
+	  </link>
+	 <joint name="torso" type="fixed">
+	    <parent link="HipsLink"/>
+	    <child link="TorsoLink"/>
+	    <origin rpy="0.0 0.0 0.0" xyz="-0.0 0.0 0.0"/>
+	 </joint>
+	 <joint name="Head_0" type="fixed">
+	    <parent link="TorsoLink"/>
+	    <child link="HeadLink"/>
+	    <origin rpy="0.0 0.0 0.0" xyz="-0.025 0.0 0.525"/>
+	 </joint>
+	 <joint name="LLeg_0" type="fixed">
+	    <parent link="HipsLink"/>
+	    <child link="LLegLink"/>
+	    <origin rpy="0.1 -0.2 0.0" xyz="-0.0 0.1 -0.15"/>
+	  </joint>
+	  <joint name="LShin_0" type="fixed">
+	    <parent link="LLegLink"/>
+	    <child link="LShinLink"/>
+	    <origin rpy="-0.13 0.2 0.0" xyz="-0.025 0.0 -0.35"/>
+	  </joint>
+	  <joint name="LAnkle_0" type="fixed">
+	    <parent link="LShinLink"/>
+	    <child link="LAnkleLink"/>
+	    <origin rpy="0.0 0.0 0.0" xyz="-0.025 0.0 -0.375"/>
+	  </joint>
+	  <joint name="RLeg_0" type="fixed">
+	    <parent link="HipsLink"/>
+	    <child link="RLegLink"/>
+	    <origin rpy="-0.1 -0.2 0.0" xyz="-0.0 -0.1 -0.15"/>
+	  </joint>
+	  <joint name="RShin_0" type="fixed">
+	    <parent link="RLegLink"/>
+	    <child link="RShinLink"/>
+	    <origin rpy="0.13 0.2 0.0" xyz="-0.025 0.0 -0.35"/>
+	  </joint>
+	  <joint name="RAnkle_0" type="fixed">
+	    <parent link="RShinLink"/>
+	    <child link="RAnkleLink"/>
+	    <origin rpy="0.0 0.0 0.0" xyz="-0.025 0.0 -0.375"/>
+	  </joint>
+	  <joint name="LArm_0" type="fixed">
+	    <parent link="TorsoLink"/>
+	    <child link="LArmLink"/>
+	    <origin rpy="-1 0.0 0.0" xyz="-0.05 0.15 0.35"/>
+	  </joint>
+	  <joint name="LElbow" type="fixed">
+	    <parent link="LArmLink"/>
+	    <child link="LElbowLink"/>
+	    <origin rpy="0 0.0 -0.2" xyz="-0.0 0.2 0.0"/>
+	  </joint>
+	  <joint name="LForearm" type="fixed">
+	    <parent link="LElbowLink"/>
+	    <child link="LForearmLink"/>
+	    <origin rpy="-0.2 0.0 0.0" xyz="-0.01 0.05 0.0"/>
+	  </joint>
+	  <joint name="LWrist_0" type="fixed">
+	    <parent link="LForearmLink"/>
+	    <child link="LHandLink"/>
+	    <origin rpy="0.0 0.0 0.0" xyz="0.01 0.24 -0.01"/>
+	  </joint>
+	 <joint name="RArm_0" type="fixed">
+	    <parent link="TorsoLink"/>
+	    <child link="RArmLink"/>
+	    <origin rpy="1 0.0 0.0" xyz="-0.05 -0.15 0.35"/>
+	  </joint>
+	  <joint name="RElbow" type="fixed">
+	    <parent link="RArmLink"/>
+	    <child link="RElbowLink"/>
+	    <origin rpy="0 0.0 0.2" xyz="0.0 -0.2 0.0"/>
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