Commit message: updated name of description package for qolo human

File: objects_descriptions/urdf/qolo_human.urdf.xacro (robot description, xacro)
@@ -1,5 +1,5 @@
 <?xml version="1.0"?>
-<robot name="qolo" xmlns:xacro="http://wiki.ros.org/xacro">
-    <xacro:arg name="prefix" default="qolo_"/>
+<robot name="qolo_human" xmlns:xacro="http://wiki.ros.org/xacro">
+    <xacro:arg name="prefix" default="qolo_human_"/>
     <xacro:arg name="connected_to" default=""/>
     <xacro:arg name="xyz" default="'0 0 0'"/>
@@ -7,6 +7,6 @@
     <xacro:arg name="mass" default="3.0"/>
     <xacro:arg name="fixed" default="1"/>
-    <xacro:include filename="$(find objects_descriptions)/urdf/qolo.xacro"/>
-    <xacro:qolo prefix="$(arg prefix)" connected_to="$(arg connected_to)" xyz="$(arg xyz)" rpy="$(arg rpy)"
+    <xacro:include filename="$(find objects_descriptions)/urdf/qolo_human.xacro"/>
+    <xacro:qolo_human prefix="$(arg prefix)" connected_to="$(arg connected_to)" xyz="$(arg xyz)" rpy="$(arg rpy)"
                  mass="$(arg mass)" fixed="$(arg fixed)"/>
 </robot>

File: objects_descriptions/urdf/qolo_human.xacro (robot description, xacro)
@@ -1,6 +1,6 @@
 <?xml version="1.0"?>
-<robot name="qolo_sim" xmlns:xacro="http://wiki.ros.org/xacro">
-    <xacro:macro name="qolo"
-                 params="prefix='qolo_' connected_to:='' xyz:='0 0 0' rpy:='0 0 0' mass=3.0, fixed:=1">
+<robot name="qolo_human_sim" xmlns:xacro="http://wiki.ros.org/xacro">
+    <xacro:macro name="qolo_human"
+                 params="prefix='qolo_human_' connected_to:='' xyz:='0 0 0' rpy:='0 0 0' mass=3.0, fixed:=1">
         <material name="gray">
             <color rgba="0.7 0.7 0.7 1"/>
