Commit message: tuning wall coloring

File: objects_descriptions/urdf/wall.xacro (robot description, xacro)
@@ -3,6 +3,9 @@
     <xacro:macro name="wall"
                  params="prefix='wall_' connected_to:='' xyz:='0 0 0' rpy:='0 0 0' mass=3.0, fixed:=1 dim:='12 0.1 1' ">
-        <material name="grey">
+        <!-- <material name="grey">
             <color rgba="0.5 0.5 0.5 1"/>
+        </material> -->
+        <material name="white">
+            <color rgba="1.0 1.0 1.0 1"/>
         </material>
         <xacro:if value="${fixed == 1}">
@@ -29,5 +32,5 @@
                     <box size="${dim}"/>
                 </geometry>
-                <material name="grey"/>
+                <material name="white"/>
             </visual>
             <collision>
